File: Eagle Files/T-ShirtPress Schematic.sch (EAGLE design)
At the start: 8 parts, among them IC1 STM32F429ZIT6

Commit message: Updated schematic
Parts:
- added C5, C6: 20pF, rcl:C-EUC1206
- added X1: 8MHz, crystal:CRYSTALHC49S
Connections:
- new net OSC_IN: C6.1, X1.1
- new net OSC_OUT: C5.1, X1.2
- net GND: now also C5.2, C6.2
Changed lines of the file:
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@@
 <part name="AC-IN" library="con-molex" library_urn="urn:adsk.eagle:library:165" deviceset="22-23-2021" device="" package3d_urn="urn:adsk.eagle:package:8078633/1"/>
 <part name="IC1" library="SamacSys_Parts" deviceset="STM32F429ZIT6" device=""/>
+<part name="X1" library="crystal" library_urn="urn:adsk.eagle:library:204" deviceset="CRYSTAL" device="HC49S" package3d_urn="urn:adsk.eagle:package:12071/1" value="8MHz"/>
+<part name="C5" library="rcl" library_urn="urn:adsk.eagle:library:334" deviceset="C-EU" device="C1206" package3d_urn="urn:adsk.eagle:package:23618/2" value="20pF"/>
+<part name="C6" library="rcl" library_urn="urn:adsk.eagle:library:334" deviceset="C-EU" device="C1206" package3d_urn="urn:adsk.eagle:package:23618/2" value="20pF"/>
 </parts>
 <sheets>
@@
 <attribute name="NAME" x="135.89" y="220.98" size="1.778" layer="95" align="center-left"/>
 <attribute name="VALUE" x="135.89" y="218.44" size="1.778" layer="96" align="center-left"/>
+</instance>
+<instance part="X1" gate="G$1" x="71.12" y="45.72" smashed="yes">
+<attribute name="NAME" x="73.66" y="46.736" size="1.778" layer="95"/>
+<attribute name="VALUE" x="73.66" y="43.18" size="1.778" layer="96"/>
+</instance>
+<instance part="C5" gate="G$1" x="76.2" y="38.1" smashed="yes">
+<attribute name="NAME" x="77.724" y="38.481" size="1.778" layer="95"/>
+<attribute name="VALUE" x="77.724" y="33.401" size="1.778" layer="96"/>
+</instance>
+<instance part="C6" gate="G$1" x="66.04" y="38.1" smashed="yes">
+<attribute name="NAME" x="67.564" y="38.481" size="1.778" layer="95"/>
+<attribute name="VALUE" x="67.564" y="33.401" size="1.778" layer="96"/>
 </instance>
 </instances>
@@
 <label x="347.98" y="205.74" size="1.778" layer="95" rot="R180" xref="yes"/>
 </segment>
+<segment>
+<pinref part="C6" gate="G$1" pin="2"/>
+<wire x1="66.04" y1="33.02" x2="66.04" y2="30.48" width="0.1524" layer="91"/>
+<pinref part="C5" gate="G$1" pin="2"/>
+<wire x1="66.04" y1="30.48" x2="71.12" y2="30.48" width="0.1524" layer="91"/>
+<wire x1="71.12" y1="30.48" x2="76.2" y2="30.48" width="0.1524" layer="91"/>
+<wire x1="76.2" y1="30.48" x2="76.2" y2="33.02" width="0.1524" layer="91"/>
+<wire x1="71.12" y1="30.48" x2="71.12" y2="27.94" width="0.1524" layer="91"/>
+<junction x="71.12" y="30.48"/>
+<label x="71.12" y="27.94" size="1.778" layer="95" rot="R270" xref="yes"/>
+</segment>
 </net>
 <net name="N$5" class="0">
@@
 </segment>
 </net>
+<net name="OSC_IN" class="0">
+<segment>
+<pinref part="X1" gate="G$1" pin="1"/>
+<wire x1="68.58" y1="45.72" x2="66.04" y2="45.72" width="0.1524" layer="91"/>
+<wire x1="66.04" y1="45.72" x2="66.04" y2="40.64" width="0.1524" layer="91"/>
+<pinref part="C6" gate="G$1" pin="1"/>
+<wire x1="66.04" y1="45.72" x2="66.04" y2="48.26" width="0.1524" layer="91"/>
+<junction x="66.04" y="45.72"/>
+<label x="66.04" y="48.26" size="1.778" layer="95" rot="R90" xref="yes"/>
+</segment>
+</net>
+<net name="OSC_OUT" class="0">
+<segment>
+<pinref part="X1" gate="G$1" pin="2"/>
+<wire x1="73.66" y1="45.72" x2="76.2" y2="45.72" width="0.1524" layer="91"/>
+<wire x1="76.2" y1="45.72" x2="76.2" y2="40.64" width="0.1524" layer="91"/>
+<pinref part="C5" gate="G$1" pin="1"/>
+<junction x="76.2" y="45.72"/>
+<wire x1="76.2" y1="45.72" x2="76.2" y2="48.26" width="0.1524" layer="91"/>
+<label x="76.2" y="48.26" size="1.778" layer="95" rot="R90" xref="yes"/>
+</segment>
+</net>

Commit message: More Schematic updates
Just working on the schematic. Trying to double check all the power electronics. Will likely get design looked over by a peer after it is designed.
Parts:
- added C10, C11, C7, C8, C9: 100nF, rcl:C-EUC1206
- SV1: value (none) -> ST-Link
Connections:
- net GND: now also C10.2, C11.2, C7.2, C8.2, C9.2
- net OSC_IN: now also IC1.PC14
- net OSC_OUT: now also IC1.PC15
- net VDD: now also C10.1, C11.1, C7.1, C8.1, C9.1
Changed lines of the file:
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@@
 <part name="C4" library="rcl" library_urn="urn:adsk.eagle:library:334" deviceset="C-EU" device="C1206" package3d_urn="urn:adsk.eagle:package:23618/2" value="100nF"/>
 <part name="PS1" library="SamacSys_Parts" deviceset="IRM-01-5" device=""/>
-<part name="SV1" library="con-lstb" library_urn="urn:adsk.eagle:library:162" deviceset="MA04-1" device="" package3d_urn="urn:adsk.eagle:package:8337/1"/>
+<part name="SV1" library="con-lstb" library_urn="urn:adsk.eagle:library:162" deviceset="MA04-1" device="" package3d_urn="urn:adsk.eagle:package:8337/1" value="ST-Link"/>
 <part name="AC-IN" library="con-molex" library_urn="urn:adsk.eagle:library:165" deviceset="22-23-2021" device="" package3d_urn="urn:adsk.eagle:package:8078633/1"/>
 <part name="IC1" library="SamacSys_Parts" deviceset="STM32F429ZIT6" device=""/>
@@
 <part name="C5" library="rcl" library_urn="urn:adsk.eagle:library:334" deviceset="C-EU" device="C1206" package3d_urn="urn:adsk.eagle:package:23618/2" value="20pF"/>
 <part name="C6" library="rcl" library_urn="urn:adsk.eagle:library:334" deviceset="C-EU" device="C1206" package3d_urn="urn:adsk.eagle:package:23618/2" value="20pF"/>
+<part name="C7" library="rcl" library_urn="urn:adsk.eagle:library:334" deviceset="C-EU" device="C1206" package3d_urn="urn:adsk.eagle:package:23618/2" value="100nF"/>
+<part name="C8" library="rcl" library_urn="urn:adsk.eagle:library:334" deviceset="C-EU" device="C1206" package3d_urn="urn:adsk.eagle:package:23618/2" value="100nF"/>
+<part name="C9" library="rcl" library_urn="urn:adsk.eagle:library:334" deviceset="C-EU" device="C1206" package3d_urn="urn:adsk.eagle:package:23618/2" value="100nF"/>
+<part name="C10" library="rcl" library_urn="urn:adsk.eagle:library:334" deviceset="C-EU" device="C1206" package3d_urn="urn:adsk.eagle:package:23618/2" value="100nF"/>
+<part name="C11" library="rcl" library_urn="urn:adsk.eagle:library:334" deviceset="C-EU" device="C1206" package3d_urn="urn:adsk.eagle:package:23618/2" value="100nF"/>
 </parts>
 <sheets>
@@
 </instance>
 <instance part="SV1" gate="1" x="358.14" y="210.82" smashed="yes" rot="R180">
-<attribute name="VALUE" x="359.41" y="220.98" size="1.778" layer="96" rot="R180"/>
+<attribute name="VALUE" x="361.95" y="220.98" size="1.778" layer="96" rot="R180"/>
 <attribute name="NAME" x="359.41" y="204.978" size="1.778" layer="95" rot="R180"/>
 </instance>
@@
 <attribute name="NAME" x="67.564" y="38.481" size="1.778" layer="95"/>
 <attribute name="VALUE" x="67.564" y="33.401" size="1.778" layer="96"/>
+</instance>
+<instance part="C7" gate="G$1" x="215.9" y="241.3" smashed="yes">
+<attribute name="NAME" x="217.424" y="241.681" size="1.778" layer="95"/>
+<attribute name="VALUE" x="217.424" y="236.601" size="1.778" layer="96"/>
+</instance>
+<instance part="C8" gate="G$1" x="226.06" y="241.3" smashed="yes">
+<attribute name="NAME" x="227.584" y="241.681" size="1.778" layer="95"/>
+<attribute name="VALUE" x="227.584" y="236.601" size="1.778" layer="96"/>
+</instance>
+<instance part="C9" gate="G$1" x="236.22" y="241.3" smashed="yes">
+<attribute name="NAME" x="237.744" y="241.681" size="1.778" layer="95"/>
+<attribute name="VALUE" x="237.744" y="236.601" size="1.778" layer="96"/>
+</instance>
+<instance part="C10" gate="G$1" x="246.38" y="241.3" smashed="yes">
+<attribute name="NAME" x="247.904" y="241.681" size="1.778" layer="95"/>
+<attribute name="VALUE" x="247.904" y="236.601" size="1.778" layer="96"/>
+</instance>
+<instance part="C11" gate="G$1" x="256.54" y="241.3" smashed="yes">
+<attribute name="NAME" x="258.064" y="241.681" size="1.778" layer="95"/>
+<attribute name="VALUE" x="258.064" y="236.601" size="1.778" layer="96"/>
 </instance>
 </instances>
@@
 <junction x="175.26" y="243.84"/>
 <label x="175.26" y="246.38" size="1.778" layer="95" rot="R90" xref="yes"/>
+<pinref part="C7" gate="G$1" pin="1"/>
+<wire x1="205.74" y1="243.84" x2="215.9" y2="243.84" width="0.1524" layer="91"/>
+<junction x="205.74" y="243.84"/>
+<pinref part="C8" gate="G$1" pin="1"/>
+<wire x1="226.06" y1="243.84" x2="215.9" y2="243.84" width="0.1524" layer="91"/>
+<junction x="215.9" y="243.84"/>
+<pinref part="C9" gate="G$1" pin="1"/>
+<wire x1="226.06" y1="243.84" x2="236.22" y2="243.84" width="0.1524" layer="91"/>
+<junction x="226.06" y="243.84"/>
+<pinref part="C10" gate="G$1" pin="1"/>
+<wire x1="236.22" y1="243.84" x2="246.38" y2="243.84" width="0.1524" layer="91"/>
+<junction x="236.22" y="243.84"/>
+<pinref part="C11" gate="G$1" pin="1"/>
+<wire x1="246.38" y1="243.84" x2="256.54" y2="243.84" width="0.1524" layer="91"/>
+<junction x="246.38" y="243.84"/>
 </segment>
 <segment>
@@
 </net>
 <net name="GND" class="0">
-<segment>
-<pinref part="C4" gate="G$1" pin="2"/>
-<pinref part="C3" gate="G$1" pin="2"/>
-<wire x1="205.74" y1="236.22" x2="195.58" y2="236.22" width="0.1524" layer="91"/>
-<pinref part="C2" gate="G$1" pin="2"/>
-<wire x1="195.58" y1="236.22" x2="185.42" y2="236.22" width="0.1524" layer="91"/>
-<junction x="195.58" y="236.22"/>
-<pinref part="C1" gate="G$1" pin="2"/>
-<wire x1="185.42" y1="236.22" x2="175.26" y2="236.22" width="0.1524" layer="91"/>
-<junction x="185.42" y="236.22"/>
-<wire x1="175.26" y1="236.22" x2="175.26" y2="233.68" width="0.1524" layer="91"/>
-<junction x="175.26" y="236.22"/>
-<label x="175.26" y="233.68" size="1.778" layer="95" rot="R270" xref="yes"/>
-</segment>
 <segment>
 <pinref part="SV1" gate="1" pin="4"/>
@@
 <label x="71.12" y="27.94" size="1.778" layer="95" rot="R270" xref="yes"/>
 </segment>
+<segment>
+<pinref part="C3" gate="G$1" pin="2"/>
+<pinref part="C2" gate="G$1" pin="2"/>
+<wire x1="195.58" y1="236.22" x2="185.42" y2="236.22" width="0.1524" layer="91"/>
+<pinref part="C1" gate="G$1" pin="2"/>
+<wire x1="185.42" y1="236.22" x2="175.26" y2="236.22" width="0.1524" layer="91"/>
+<junction x="185.42" y="236.22"/>
+<wire x1="175.26" y1="236.22" x2="175.26" y2="233.68" width="0.1524" layer="91"/>
+<junction x="175.26" y="236.22"/>
+<label x="175.26" y="233.68" size="1.778" layer="95" rot="R270" xref="yes"/>
+<pinref part="C4" gate="G$1" pin="2"/>
+<wire x1="195.58" y1="236.22" x2="205.74" y2="236.22" width="0.1524" layer="91"/>
+<junction x="195.58" y="236.22"/>
+<pinref part="C7" gate="G$1" pin="2"/>
+<wire x1="205.74" y1="236.22" x2="215.9" y2="236.22" width="0.1524" layer="91"/>
+<junction x="205.74" y="236.22"/>
+<pinref part="C8" gate="G$1" pin="2"/>
+<wire x1="215.9" y1="236.22" x2="226.06" y2="236.22" width="0.1524" layer="91"/>
+<junction x="215.9" y="236.22"/>
+<pinref part="C9" gate="G$1" pin="2"/>
+<wire x1="226.06" y1="236.22" x2="236.22" y2="236.22" width="0.1524" layer="91"/>
+<junction x="226.06" y="236.22"/>
+<pinref part="C10" gate="G$1" pin="2"/>
+<wire x1="236.22" y1="236.22" x2="246.38" y2="236.22" width="0.1524" layer="91"/>
+<junction x="236.22" y="236.22"/>
+<pinref part="C11" gate="G$1" pin="2"/>
+<wire x1="246.38" y1="236.22" x2="256.54" y2="236.22" width="0.1524" layer="91"/>
+<junction x="246.38" y="236.22"/>
+</segment>
 </net>
 <net name="N$5" class="0">
@@
 <label x="66.04" y="48.26" size="1.778" layer="95" rot="R90" xref="yes"/>
 </segment>
+<segment>
+<pinref part="IC1" gate="G$1" pin="PC14"/>
+<wire x1="35.56" y1="185.42" x2="22.86" y2="185.42" width="0.1524" layer="91"/>
+<wire x1="22.86" y1="185.42" x2="22.86" y2="187.96" width="0.1524" layer="91"/>
+<wire x1="22.86" y1="187.96" x2="20.32" y2="187.96" width="0.1524" layer="91"/>
+<label x="20.32" y="187.96" size="1.778" layer="95" rot="R180" xref="yes"/>
+</segment>
 </net>
 <net name="OSC_OUT" class="0">
@@
 <label x="76.2" y="48.26" size="1.778" layer="95" rot="R90" xref="yes"/>
 </segment>
-</net>
+<segment>
+<pinref part="IC1" gate="G$1" pin="PC15"/>
+<wire x1="35.56" y1="182.88" x2="22.86" y2="182.88" width="0.1524" layer="91"/>
+<wire x1="22.86" y1="182.88" x2="22.86" y2="180.34" width="0.1524" layer="91"/>
+<wire x1="22.86" y1="180.34" x2="20.32" y2="180.34" width="0.1524" layer="91"/>
+<label x="20.32" y="180.34" size="1.778" layer="95" rot="R180" xref="yes"/>
+</segment>
+</net>

Commit message: Enabled SWD and updated symbols on schematic
Parts:
- removed SV1: ST-Link, con-lstb:MA04-1
- added JP1: (no value), pinhead:PINHD-1X5
- AC-IN: value 22-23-2021 -> (none); device con-molex:22-23-2021 -> pinhead:PINHD-1X2
Connections:
- new net N$1: JP1.4
- net GND: now also JP1.5; no longer SV1.4
- net N$5: now also JP1.2; no longer SV1.2
- net N$6: now also JP1.3; no longer SV1.3
- net OSC_IN: now also IC1.PH0; no longer IC1.PC14
- net OSC_OUT: now also IC1.PH1; no longer IC1.PC15
- net VDD: now also JP1.1; no longer SV1.1
- net VLINE: now also AC-IN.2; no longer AC-IN-1.S
- net VNEUTRAL: now also AC-IN.1; no longer AC-IN-2.S
